File: hackpad_proto.kicad_sch (KiCad schematic)
At the start: 40 parts, among them J1 Conn_01x04, SW1 SW_Push, SW10 SW_Push, SW11 SW_Push, SW12 SW_Push, SW13 RotaryEncoder_Switch, SW2 SW_Push, SW3 SW_Push, SW4 SW_Push, SW5 SW_Push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

Commit message: Updated NostPad hardware design layout
Parts:
- D13, D14, D15, D16, D17, D18, D19, D20, D21, D22, D23, D24: footprint LED_SMD:LED_SK6812_PLCC4_5.0x5.0mm_P3.2mm -> footprints:SK6812MINI-E_fixed
Changed lines of the file:
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@@
 			)
 		)
-		(property "Footprint" "LED_SMD:LED_SK6812_PLCC4_5.0x5.0mm_P3.2mm"
+		(property "Footprint" "footprints:SK6812MINI-E_fixed"
 			(at 48.26 71.12 0)
 			(hide yes)
@@
 			)
 		)
-		(property "Footprint" "LED_SMD:LED_SK6812_PLCC4_5.0x5.0mm_P3.2mm"
+		(property "Footprint" "footprints:SK6812MINI-E_fixed"
 			(at 181.61 71.12 0)
 			(hide yes)
@@
 			)
 		)
-		(property "Footprint" "LED_SMD:LED_SK6812_PLCC4_5.0x5.0mm_P3.2mm"
+		(property "Footprint" "footprints:SK6812MINI-E_fixed"
 			(at 162.56 71.12 0)
 			(hide yes)
@@
 			)
 		)
-		(property "Footprint" "LED_SMD:LED_SK6812_PLCC4_5.0x5.0mm_P3.2mm"
+		(property "Footprint" "footprints:SK6812MINI-E_fixed"
 			(at 124.46 71.12 0)
 			(hide yes)
@@
 			)
 		)
-		(property "Footprint" "LED_SMD:LED_SK6812_PLCC4_5.0x5.0mm_P3.2mm"
+		(property "Footprint" "footprints:SK6812MINI-E_fixed"
 			(at 143.51 71.12 0)
 			(hide yes)
@@
 			)
 		)
-		(property "Footprint" "LED_SMD:LED_SK6812_PLCC4_5.0x5.0mm_P3.2mm"
+		(property "Footprint" "footprints:SK6812MINI-E_fixed"
 			(at 86.36 71.12 0)
 			(hide yes)
@@
 			)
 		)
-		(property "Footprint" "LED_SMD:LED_SK6812_PLCC4_5.0x5.0mm_P3.2mm"
+		(property "Footprint" "footprints:SK6812MINI-E_fixed"
 			(at 67.31 71.12 0)
 			(hide yes)
@@
 			)
 		)
-		(property "Footprint" "LED_SMD:LED_SK6812_PLCC4_5.0x5.0mm_P3.2mm"
+		(property "Footprint" "footprints:SK6812MINI-E_fixed"
 			(at 218.44 71.12 0)
 			(hide yes)
@@
 			)
 		)
-		(property "Footprint" "LED_SMD:LED_SK6812_PLCC4_5.0x5.0mm_P3.2mm"
+		(property "Footprint" "footprints:SK6812MINI-E_fixed"
 			(at 199.39 71.12 0)
 			(hide yes)
@@
 			)
 		)
-		(property "Footprint" "LED_SMD:LED_SK6812_PLCC4_5.0x5.0mm_P3.2mm"
+		(property "Footprint" "footprints:SK6812MINI-E_fixed"
 			(at 256.54 71.12 0)
 			(hide yes)
@@
 			)
 		)
-		(property "Footprint" "LED_SMD:LED_SK6812_PLCC4_5.0x5.0mm_P3.2mm"
+		(property "Footprint" "footprints:SK6812MINI-E_fixed"
 			(at 237.49 71.12 0)
 			(hide yes)
@@
 			)
 		)
-		(property "Footprint" "LED_SMD:LED_SK6812_PLCC4_5.0x5.0mm_P3.2mm"
+		(property "Footprint" "footprints:SK6812MINI-E_fixed"
 			(at 105.41 71.12 0)
 			(hide yes)
